Commit message: ignore odom frame and add velodyne frame

File: xacro/modelc.xacro (robot description, xacro)
@@ -169,4 +169,11 @@
         <child link="imu"/>
     </joint>
+    <link name="velodyne">
+    </link>
+    <joint name="velodyne" type="fixed">
+        <origin xyz="0 0 1.0" rpy="0 0 0"/>
+        <parent link="base_link"/>
+        <child link="velodyne"/>
+    </joint>
     <!-- ===============  Transmission =============== -->
     <transmission name="right_wheel_trans">
